Commit message: controllers-close

File: go1_ros2/src/go1_description/xacro/leg.xacro (robot description, xacro)
@@ -27,4 +27,14 @@
             </xacro:if>
         </joint>
+          <ros2_control name="${name}_hip" type="system">
+	    <hardware>
+	      <plugin>gazebo_ros2_control/GazeboSystem</plugin>
+	    </hardware>
+	    <joint name="${name}_hip_joint">
+	      <command_interface name="effort"/>
+	      <state_interface name="position"/>
+	      <state_interface name="velocity"/>
+	    </joint>
+	  </ros2_control>
         <joint name="${name}_hip_rotor_joint" type="fixed">
             <xacro:if value="${(mirror_dae == False) and (front_hind_dae == True)}">
@@ -108,4 +118,14 @@
             <limit effort="${thigh_torque_max}" velocity="${thigh_velocity_max}" lower="${thigh_position_min}" upper="${thigh_position_max}"/>
         </joint>
+          <ros2_control name="${name}_thigh" type="system">
+	    <hardware>
+	      <plugin>gazebo_ros2_control/GazeboSystem</plugin>
+	    </hardware>
+	    <joint name="${name}_thigh_joint">
+	      <command_interface name="effort"/>
+	      <state_interface name="position"/>
+	      <state_interface name="velocity"/>
+	    </joint>
+	  </ros2_control>
         <joint name="${name}_thigh_rotor_joint" type="fixed">
             <origin rpy="0 0 0" xyz="${thigh_rotor_offset_x} ${thigh_rotor_offset_y*mirror} 0"/>
@@ -172,4 +192,14 @@
             <limit effort="${calf_torque_max}" velocity="${calf_velocity_max}" lower="${calf_position_min}" upper="${calf_position_max}"/>
         </joint>
+        <ros2_control name="${name}_calf" type="system">
+	    <hardware>
+	      <plugin>gazebo_ros2_control/GazeboSystem</plugin>
+	    </hardware>
+	    <joint name="${name}_calf_joint">
+	      <command_interface name="effort"/>
+	      <state_interface name="position"/>
+	      <state_interface name="velocity"/>
+	    </joint>
+	  </ros2_control>
         <joint name="${name}_calf_rotor_joint" type="fixed">
             <origin rpy="0 0 0" xyz="${calf_rotor_offset_x} ${calf_rotor_offset_y*mirror} 0"/>
