Commit message: updated-base-link

File: go1_ros2/src/go1_description/xacro/gazebo.xacro (robot description, xacro)
@@ -6,5 +6,5 @@
             <remapping>odom:=odom/ground_truth</remapping>
         </ros>
-        <body_name>base</body_name>
+        <body_name>base_link</body_name>
         <frame_name>world</frame_name>
         <update_rate>10.0</update_rate>
@@ -25,5 +25,5 @@
             <frequency>10</frequency>
             <plot>
-                <link>base</link>
+                <link>base_link</link>
                 <pose>0 0 0 0 0 0</pose>
                 <material>Gazebo/Yellow</material>
@@ -323,5 +323,5 @@
         </visual>
     </gazebo>
-    <gazebo reference="base">
+    <gazebo reference="base_link">
         <material>Gazebo/Green</material>
         <turnGravityOff>false</turnGravityOff>

File: go1_ros2/src/go1_description/xacro/robot.xacro (robot description, xacro)
@@ -19,8 +19,8 @@
             <origin rpy="0 0 0" xyz="0 0 0"/>
             <parent link="world"/>
-            <child link="base"/>
+            <child link="base_link"/>
         </joint>
     </xacro:if>
-    <link name="base">
+    <link name="base_link">
         <visual>
             <origin rpy="0 0 0" xyz="0 0 0"/>
@@ -32,5 +32,5 @@
     <joint name="floating_base" type="fixed">
         <origin rpy="0 0 0" xyz="0 0 0"/>
-        <parent link="base"/>
+        <parent link="base_link"/>
         <child link="trunk"/>
     </joint>

Commit message: getting-close

File: go1_ros2/src/go1_description/xacro/gazebo.xacro (robot description, xacro)
@@ -249,78 +249,4 @@
     </sensor>
   </gazebo>
-    <!-- Foot contacts. -->
-    <gazebo reference="FR_calf">
-        <sensor name="FR_foot_contact" type="contact">
-        <update_rate>100</update_rate>
-        <!--
-        <plugin name="contactPlugin" filename="libunitreeFootContactPlugin.so"/>-->
-        <contact>
-            <collision>FR_calf_fixed_joint_lump__FR_foot_collision_1</collision>
-        </contact>
-        </sensor>
-    </gazebo>
-    <gazebo reference="FL_calf">
-        <sensor name="FL_foot_contact" type="contact">
-        <update_rate>100</update_rate>
-        <!--
-        <plugin name="contactPlugin" filename="libunitreeFootContactPlugin.so"/>-->
-        <contact>
-            <collision>FL_calf_fixed_joint_lump__FL_foot_collision_1</collision>
-        </contact>
-        </sensor>
-    </gazebo>
-    <gazebo reference="RR_calf">
-        <sensor name="RR_foot_contact" type="contact">
-        <update_rate>100</update_rate>
-        <!--
-        <plugin name="contactPlugin" filename="libunitreeFootContactPlugin.so"/>-->
-        <contact>
-            <collision>RR_calf_fixed_joint_lump__RR_foot_collision_1</collision>
-        </contact>
-        </sensor>
-    </gazebo>
-    <gazebo reference="RL_calf">
-        <sensor name="RL_foot_contact" type="contact">
-        <update_rate>100</update_rate>
-        <!--
-        <plugin name="contactPlugin" filename="libunitreeFootContactPlugin.so"/>--> s
-        <contact>
-            <collision>RL_calf_fixed_joint_lump__RL_foot_collision_1</collision>
-        </contact>
-        </sensor>
-    </gazebo>
-    <!-- Visualization of Foot contacts. -->
-    <gazebo reference="FR_foot">
-        <visual>
-        <!--
-            <plugin name="drawForcePlugin" filename="libunitreeDrawForcePlugin.so">
-                <topicName>FR_foot_contact</topicName>
-            </plugin>-->
-        </visual>
-    </gazebo>
-    <gazebo reference="FL_foot">
-        <visual>
-        <!--
-            <plugin name="drawForcePlugin" filename="libunitreeDrawForcePlugin.so">
-                <topicName>FL_foot_contact</topicName>
-            </plugin>-->
-        </visual>
-    </gazebo>
-    <gazebo reference="RR_foot">
-        <visual>
-        <!--
-            <plugin name="drawForcePlugin" filename="libunitreeDrawForcePlugin.so">
-                <topicName>RR_foot_contact</topicName>
-            </plugin>-->
-        </visual>
-    </gazebo>
-    <gazebo reference="RL_foot">
-        <visual>
-        <!--
-            <plugin name="drawForcePlugin" filename="libunitreeDrawForcePlugin.so">
-                <topicName>RL_foot_contact</topicName>
-            </plugin>-->
-        </visual>
-    </gazebo>
     <gazebo reference="base_link">
         <material>Gazebo/Green</material>
@@ -344,18 +270,18 @@
     </gazebo>
     <!-- FL leg -->
-    <gazebo reference="FL_hip">
-        <mu1>0.2</mu1>
-        <mu2>0.2</mu2>
-        <material>Gazebo/DarkGrey</material>
-    </gazebo>
-    <gazebo reference="FL_thigh">
-        <mu1>0.2</mu1>
-        <mu2>0.2</mu2>
-        <self_collide>1</self_collide>
-        <material>Gazebo/DarkGrey</material>
-        <kp  value="1000000.0"/>
-        <kd  value="1.0"/>
-    </gazebo>
-    <gazebo reference="FL_calf">
+    <gazebo reference="lf_hip_link">
+        <mu1>0.2</mu1>
+        <mu2>0.2</mu2>
+        <material>Gazebo/DarkGrey</material>
+    </gazebo>
+    <gazebo reference="lf_upper_leg_link">
+        <mu1>0.2</mu1>
+        <mu2>0.2</mu2>
+        <self_collide>1</self_collide>
+        <material>Gazebo/DarkGrey</material>
+        <kp  value="1000000.0"/>
+        <kd  value="1.0"/>
+    </gazebo>
+    <gazebo reference="lf_lower_leg_link">
         <mu1>0.2</mu1>
         <mu2>0.2</mu2>
@@ -371,23 +297,23 @@
     </gazebo>
     <!-- FR leg -->
-    <gazebo reference="FR_hip">
-        <mu1>0.2</mu1>
-        <mu2>0.2</mu2>
-        <material>Gazebo/DarkGrey</material>
-    </gazebo>
-    <gazebo reference="FR_thigh">
-        <mu1>0.2</mu1>
-        <mu2>0.2</mu2>
-        <self_collide>1</self_collide>
-        <material>Gazebo/DarkGrey</material>
-        <kp  value="1000000.0"/>
-        <kd  value="1.0"/>
-    </gazebo>
-    <gazebo reference="FR_calf">
-        <mu1>0.2</mu1>
-        <mu2>0.2</mu2>
-        <self_collide>1</self_collide>
-    </gazebo>
-    <gazebo reference="FR_foot">
+    <gazebo reference="rf_hip">
+        <mu1>0.2</mu1>
+        <mu2>0.2</mu2>
+        <material>Gazebo/DarkGrey</material>
+    </gazebo>
+    <gazebo reference="rf_upper_leg_link">
+        <mu1>0.2</mu1>
+        <mu2>0.2</mu2>
+        <self_collide>1</self_collide>
+        <material>Gazebo/DarkGrey</material>
+        <kp  value="1000000.0"/>
+        <kd  value="1.0"/>
+    </gazebo>
+    <gazebo reference="rf_lower_leg_link">
+        <mu1>0.2</mu1>
+        <mu2>0.2</mu2>
+        <self_collide>1</self_collide>
+    </gazebo>
+    <gazebo reference="rf_foot_link">
         <mu1>0.6</mu1>
         <mu2>0.6</mu2>
@@ -398,23 +324,23 @@
     </gazebo>
     <!-- RL leg -->
-    <gazebo reference="RL_hip">
-        <mu1>0.2</mu1>
-        <mu2>0.2</mu2>
-        <material>Gazebo/DarkGrey</material>
-    </gazebo>
-    <gazebo reference="RL_thigh">
-        <mu1>0.2</mu1>
-        <mu2>0.2</mu2>
-        <self_collide>1</self_collide>
-        <material>Gazebo/DarkGrey</material>
-        <kp  value="1000000.0"/>
-        <kd  value="1.0"/>
-    </gazebo>
-    <gazebo reference="RL_calf">
-        <mu1>0.2</mu1>
-        <mu2>0.2</mu2>
-        <self_collide>1</self_collide>
-    </gazebo>
-    <gazebo reference="RL_foot">
+    <gazebo reference="lh_hip">
+        <mu1>0.2</mu1>
+        <mu2>0.2</mu2>
+        <material>Gazebo/DarkGrey</material>
+    </gazebo>
+    <gazebo reference="lh_upper_leg_link">
+        <mu1>0.2</mu1>
+        <mu2>0.2</mu2>
+        <self_collide>1</self_collide>
+        <material>Gazebo/DarkGrey</material>
+        <kp  value="1000000.0"/>
+        <kd  value="1.0"/>
+    </gazebo>
+    <gazebo reference="lh_lower_leg_link">
+        <mu1>0.2</mu1>
+        <mu2>0.2</mu2>
+        <self_collide>1</self_collide>
+    </gazebo>
+    <gazebo reference="lh_foot_link">
         <mu1>0.6</mu1>
         <mu2>0.6</mu2>
@@ -425,23 +351,23 @@
     </gazebo>
     <!-- RR leg -->
-    <gazebo reference="RR_hip">
-        <mu1>0.2</mu1>
-        <mu2>0.2</mu2>
-        <material>Gazebo/DarkGrey</material>
-    </gazebo>
-    <gazebo reference="RR_thigh">
-        <mu1>0.2</mu1>
-        <mu2>0.2</mu2>
-        <self_collide>1</self_collide>
-        <material>Gazebo/DarkGrey</material>
-        <kp  value="1000000.0"/>
-        <kd  value="1.0"/>
-    </gazebo>
-    <gazebo reference="RR_calf">
-        <mu1>0.2</mu1>
-        <mu2>0.2</mu2>
-        <self_collide>1</self_collide>
-    </gazebo>
-    <gazebo reference="RR_foot">
+    <gazebo reference="rh_hip">
+        <mu1>0.2</mu1>
+        <mu2>0.2</mu2>
+        <material>Gazebo/DarkGrey</material>
+    </gazebo>
+    <gazebo reference="rh_upper_leg_link">
+        <mu1>0.2</mu1>
+        <mu2>0.2</mu2>
+        <self_collide>1</self_collide>
+        <material>Gazebo/DarkGrey</material>
+        <kp  value="1000000.0"/>
+        <kd  value="1.0"/>
+    </gazebo>
+    <gazebo reference="rh_lower_leg_link">
+        <mu1>0.2</mu1>
+        <mu2>0.2</mu2>
+        <self_collide>1</self_collide>
+    </gazebo>
+    <gazebo reference="rh_foot_link">
         <mu1>0.6</mu1>
         <mu2>0.6</mu2>

File: go1_ros2/src/go1_description/xacro/leg.xacro (robot description, xacro)
@@ -6,5 +6,5 @@
             <xacro:insert_block name="origin"/>
             <parent link="trunk"/>
-            <child link="${name}_hip"/>
+            <child link="${name}_hip_link"/>
             <axis xyz="1 0 0"/>
             <dynamics damping="${damping}" friction="${friction}"/>
@@ -16,5 +16,5 @@
             </xacro:if>
         </joint>
-        <link name="${name}_hip">
+        <link name="${name}_hip_link">
             <visual>
                 <xacro:if value="${(mirror_dae == True) and (front_hind_dae == True)}">
@@ -52,5 +52,5 @@
         <joint name="${name}_hip_fixed" type="fixed">
             <origin rpy="0 0 0" xyz="0 ${(hip_offset)*mirror} 0"/>
-            <parent link="${name}_hip"/>
+            <parent link="${name}_hip_link"/>
             <child link="${name}_thigh_shoulder"/>
         </joint>
@@ -64,13 +64,13 @@
             </collision>
         </link>
-        <joint name="${name}_thigh_joint" type="revolute">
+        <joint name="${name}_upper_leg_joint" type="revolute">
             <origin rpy="0 0 0" xyz="0 ${thigh_offset*mirror} 0"/>
-            <parent link="${name}_hip"/>
-            <child link="${name}_thigh"/>
+            <parent link="${name}_hip_link"/>
+            <child link="${name}_upper_leg_link"/>
             <axis xyz="0 1 0"/>
             <dynamics damping="${damping}" friction="${friction}"/>
             <limit effort="${thigh_torque_max}" velocity="${thigh_velocity_max}" lower="${thigh_min*PI/180.0}" upper="${thigh_max*PI/180.0}"/>
         </joint>
-        <link name="${name}_thigh">
+        <link name="${name}_upper_leg_link">
             <visual>
                 <origin rpy="0 0 0" xyz="0 0 0"/>
@@ -100,13 +100,13 @@
             </inertial>
         </link>
-        <joint name="${name}_calf_joint" type="revolute">
+        <joint name="${name}_lower_leg_joint" type="revolute">
             <origin rpy="0 0 0" xyz="0 0 ${-thigh_length}"/>
-            <parent link="${name}_thigh"/>
-            <child link="${name}_calf"/>
+            <parent link="${name}_upper_leg_link"/>
+            <child link="${name}_lower_leg_link"/>
             <axis xyz="0 1 0"/>
             <dynamics damping="${damping}" friction="${friction}"/>
             <limit effort="${calf_torque_max}" velocity="${calf_velocity_max}" lower="${calf_min*PI/180.0}" upper="${calf_max*PI/180.0}"/>
         </joint>
-        <link name="${name}_calf">
+        <link name="${name}_lower_leg_link">
             <visual>
                 <origin rpy="0 0 0" xyz="0 0 0"/>
@@ -131,10 +131,10 @@
             </inertial>
         </link>
-        <joint name="${name}_foot_fixed" type="fixed">
+        <joint name="${name}_foot_joint" type="fixed">
             <origin rpy="0 0 0" xyz="0 0 ${-(calf_length)}"/>
-            <parent link="${name}_calf"/>
-            <child link="${name}_foot"/>
+            <parent link="${name}_lower_leg_link"/>
+            <child link="${name}_foot_link"/>
         </joint>
-        <link name="${name}_foot">
+        <link name="${name}_foot_link">
             <visual>
                 <origin rpy="0 0 0" xyz="0 0 0"/>
@@ -159,24 +159,24 @@
         </link>
         <xacro:leg_transmission name="${name}"/>
-          <ros2_control name="${name}" type="system">
-	    <hardware>
-	      <plugin>gazebo_ros2_control/GazeboSystem</plugin>
-	    </hardware>
-	    <joint name="${name}_hip_joint">
-	      <command_interface name="effort"/>
-	      <state_interface name="position"/>
-	      <state_interface name="velocity"/>
-	    </joint>
-	    <joint name="${name}_thigh_joint">
-	      <command_interface name="effort"/>
-	      <state_interface name="position"/>
-	      <state_interface name="velocity"/>
-	    </joint>
-	    <joint name="${name}_calf_joint">
-	      <command_interface name="effort"/>
-	      <state_interface name="position"/>
-	      <state_interface name="velocity"/>
-	    </joint>
-	  </ros2_control>
+        <ros2_control name="${name}" type="system">
+            <hardware>
+                <plugin>gazebo_ros2_control/GazeboSystem</plugin>
+            </hardware>
+            <joint name="${name}_hip_joint">
+                <command_interface name="effort"/>
+                <state_interface name="position"/>
+                <state_interface name="velocity"/>
+            </joint>
+            <joint name="${name}_upper_leg_joint">
+                <command_interface name="effort"/>
+                <state_interface name="position"/>
+                <state_interface name="velocity"/>
+            </joint>
+            <joint name="${name}_lower_leg_joint">
+                <command_interface name="effort"/>
+                <state_interface name="position"/>
+                <state_interface name="velocity"/>
+            </joint>
+        </ros2_control>
     </xacro:macro>
 </robot>

File: go1_ros2/src/go1_description/xacro/robot.xacro (robot description, xacro)
@@ -112,14 +112,14 @@
         </collision>
     </link>
-    <xacro:leg name="FR" mirror="-1" mirror_dae="False" front_hind="1" front_hind_dae="True">
+    <xacro:leg name="rf" mirror="-1" mirror_dae="False" front_hind="1" front_hind_dae="True">
         <origin rpy="0 0 0" xyz="${leg_offset_x} ${-leg_offset_y} 0"/>
     </xacro:leg>
-    <xacro:leg name="FL" mirror="1" mirror_dae="True" front_hind="1" front_hind_dae="True">
+    <xacro:leg name="lf" mirror="1" mirror_dae="True" front_hind="1" front_hind_dae="True">
         <origin rpy="0 0 0" xyz="${leg_offset_x} ${leg_offset_y} 0"/>
     </xacro:leg>
-    <xacro:leg name="RR" mirror="-1" mirror_dae="False" front_hind="-1" front_hind_dae="False">
+    <xacro:leg name="rh" mirror="-1" mirror_dae="False" front_hind="-1" front_hind_dae="False">
         <origin rpy="0 0 0" xyz="${-leg_offset_x} ${-leg_offset_y} 0"/>
     </xacro:leg>
-    <xacro:leg name="RL" mirror="1" mirror_dae="True" front_hind="-1" front_hind_dae="False">
+    <xacro:leg name="lh" mirror="1" mirror_dae="True" front_hind="-1" front_hind_dae="False">
         <origin rpy="0 0 0" xyz="${-leg_offset_x} ${leg_offset_y} 0"/>
     </xacro:leg>
