Commit message: fixing-obstacles-slam

File: src/unitree_ros2_sim/go1_sim/go1_description/xacro/lidar.xacro (robot description, xacro)
@@ -1,5 +1,5 @@
 <?xml version="1.0"?>
 <robot xmlns:xacro="http://www.ros.org/wiki/xacro">
-  <xacro:macro name="lidar" params="name *origin hz:=10 samples:=512 min_range:=0.1 max_range:=90 noise:=0.008">
+  <xacro:macro name="lidar" params="name *origin hz:=15 samples:=512 min_range:=0.1 max_range:=90 noise:=0.0008">
     <joint name="laser_joint" type="fixed">
       <xacro:insert_block name="origin" />

File: src/unitree_ros2_sim/go1_sim/go1_description/xacro/robot.xacro (robot description, xacro)
@@ -31,14 +31,12 @@
     <origin xyz="0 0 0.010" rpy="0 0 0"/>
   </joint>
-  -->
-  <!--
       <gazebo>
         <plugin name="p3d_ground_truth" filename="libgazebo_ros_p3d.so">
-            <body_name>base_footprint</body_name>
+            <body_name>base_link</body_name>
             <topic_name>odom</topic_name>
             <update_rate>100</update_rate>
         </plugin>
     </gazebo>
-   -->
+  -->
     <link name="base_link">
         <visual>
