Commit message: nav-last-commit-stable

File: src/unitree_ros2_sim/go1_sim/go1_description/xacro/robot.xacro (robot description, xacro)
@@ -96,5 +96,5 @@
         <geometry>
             <mesh filename="file://$(find go1_description)/meshes/mounting_frame.obj"/>
-        </geometry>
+        </geometry>s
       </visual>
       <!-- <inertial>
@@ -105,5 +105,5 @@
     </link>
     <!-- Ouster OS1-32 Lidar -->
-    <xacro:lidar name="os1_sensor" hz="10" samples="512" min_range="0.1" max_range="90" >
+    <xacro:lidar name="os1_sensor" hz="15" samples="512" min_range="0.1" max_range="90" >
         <origin xyz="0.007 0.0 0.134" rpy="0.0 0 1.5708" />
     </xacro:lidar>
