Commit message: clean-up

File: unitree-go2-ros2/robots/descriptions/go1_description/xacro/lidar.xacro (robot description, xacro)
@@ -22,4 +22,5 @@
          <origin xyz="0 0 0.0365" rpy="0 0 0" />
          <geometry>
+            <cylinder radius="0.04" length="0.073"/>
          </geometry>
       </collision>

Commit message: minor-fixes

File: unitree-go2-ros2/robots/descriptions/go1_description/xacro/lidar.xacro (robot description, xacro)
@@ -1,5 +1,5 @@
 <?xml version="1.0"?>
 <robot xmlns:xacro="http://www.ros.org/wiki/xacro">
-  <xacro:macro name="lidar" params="name *origin hz:=10 samples:=512 min_range:=0.1 max_range:=90 noise:=0.008">
+  <xacro:macro name="lidar" params="name *origin hz:=15 samples:=512 min_range:=0.1 max_range:=90 noise:=0.008">
     <joint name="lidar_joint" type="fixed">
       <xacro:insert_block name="origin" />

File: unitree-go2-ros2/robots/descriptions/go1_description/xacro/robot.xacro (robot description, xacro)
@@ -105,5 +105,5 @@
     </link>
     <!-- Ouster OS1-32 Lidar -->
-    <xacro:lidar name="os1_sensor" hz="10" samples="512" min_range="0.1" max_range="90" >
+    <xacro:lidar name="os1_sensor" hz="15" samples="512" min_range="0.1" max_range="90" >
         <origin xyz="0.007 0.0 0.134" rpy="0.0 0 1.5708" />
     </xacro:lidar>
