Commit message: ouster-fixed-frame

File: real/src/unitree_ros2/go1_description/xacro/robot.xacro (robot description, xacro)
@@ -3,7 +3,4 @@
     <xacro:arg name="DEBUG" default="false"/>
     <xacro:arg name="use_nav2_links" default="false"/>
-    <xacro:arg name="lidar_x_offset" default="0.186"/>
-    <xacro:arg name="lidar_y_offset" default="0.0"/>
-    <xacro:arg name="lidar_z_offset" default="0.225"/>
     <xacro:include filename="$(find go1_description)/xacro/const.xacro"/>
     <xacro:include filename="$(find go1_description)/xacro/materials.xacro"/>
@@ -13,4 +10,6 @@
     <xacro:include filename="$(find go1_description)/xacro/depthCamera.xacro"/>
     <xacro:include filename="$(find go1_description)/xacro/ultraSound.xacro"/>
+    <xacro:include filename="$(find go1_description)/xacro/lidar.xacro"/>
+    <xacro:include filename="$(find go1_description)/xacro/_d435i.urdf.xacro"/>
     <!-- <xacro:include filename="$(find go1_gazebo)/launch/stairs.urdf.xacro"/> -->
     <!-- <xacro:stairs stairs="15" xpos="0" ypos="0" zpos="0" /> -->
@@ -55,11 +54,4 @@
                 <axis xyz="0 0 -1" />
                 <limit effort="100000.0" lower="0.0" upper="1.0" velocity="100000.0"/>
-        </joint>
-        <link name="base_laser" />
-        <joint name="base_link_to_lidar" type="fixed">
-            <!-- TODO need to measure mounting or make this a parameter -->
-            <origin rpy="0 0 0" xyz="$(arg lidar_x_offset) $(arg lidar_y_offset) $(arg lidar_z_offset)"/>
-            <parent link="base_link"/>
-            <child link="base_laser"/>
         </joint>
     </xacro:if>
@@ -117,4 +109,32 @@
         </collision>
     </link>
+    <!-- MOUNTING FRAME -->
+    <joint name="mount_joint" type="fixed">
+        <origin xyz="0.179 0.0 0.091" rpy="0 0 0" />
+        <parent link="base_link"/>
+        <child link="mount_frame"/>
+    </joint>
+    <link name="mount_frame">
+      <visual>
+        <origin xyz="-0.252 -0.19 0.121" rpy="0 0 0" />
+        <geometry>
+            <mesh filename="file://$(find go1_description)/meshes/mounting_frame.obj"/>
+        </geometry>
+      </visual>
+      <!-- <inertial>
+         <mass value="0.033"/>
+         <origin xyz="0 0 0.091" rpy="0 0 0" />
+         <inertia ixx="0.000241148" ixy="0" ixz="0" iyy="0.000241148" iyz="0" izz="0.000264"/>
+      </inertial> -->
+    </link>
+    <!-- Ouster OS1-32 Lidar -->
+    <xacro:lidar name="os1_sensor" hz="15" samples="512" min_range="0.1" max_range="90" >
+        <origin xyz="0.007 0.0 0.134" rpy="0.0 0 3.14159" />
+    </xacro:lidar>
+    <!-- Realsense d435i Camera -->
+    <xacro:sensor_d435i parent="mount_frame" use_nominal_extrinsics="true" >
+    	<origin xyz="0.076 0.0 0.062" rpy="0 0 0" />
+    </xacro:sensor_d435i>
+    <!-- End realsense -->
     <xacro:leg name="FR" mirror="-1" mirror_dae= "False" front_hind="1"  front_hind_dae="True"  />
     <xacro:leg name="FL" mirror="1"  mirror_dae="True"   front_hind="1"  front_hind_dae="True"  />

Commit message: added-camera

File: real/src/unitree_ros2/go1_description/xacro/robot.xacro (robot description, xacro)
@@ -129,5 +129,5 @@
     </link>
     <!-- Ouster OS1-32 Lidar -->
-    <xacro:lidar name="os1_sensor" hz="15" samples="512" min_range="0.1" max_range="90" >
+    <xacro:lidar name="os1_sensor" hz="20" samples="512" min_range="0.1" max_range="90" >
         <origin xyz="0.007 0.0 0.134" rpy="0.0 0 3.14159" />
     </xacro:lidar>

File: sim/unitree-go2-ros2/robots/descriptions/go1_description/xacro/robot.xacro (robot description, xacro)
@@ -105,6 +105,6 @@
     </link>
     <!-- Ouster OS1-32 Lidar -->
-    <xacro:lidar name="os1_sensor" hz="15" samples="512" min_range="0.1" max_range="90" >
-        <origin xyz="0.007 0.0 0.134" rpy="0.0 0 1.5708" />
+    <xacro:lidar name="os1_sensor" hz="20" samples="512" min_range="0.1" max_range="90" >
+        <origin xyz="0.007 0.0 0.134" rpy="0.0 0 3.14159" />
     </xacro:lidar>
     <!-- Realsense d435i Camera -->
