Commit message: first-exp-ok

File: real/src/unitree_ros2/go1_description/xacro/_d435.urdf.xacro (robot description, xacro)
@@ -128,134 +128,4 @@
       </xacro:usb_plug>
     </xacro:if>
-    <!-- gazebo plugin -->
-    <!-- Load parameters to model's main link-->
-    <xacro:property name="deg_to_rad" value="0.01745329251994329577" />
-    <gazebo reference="${name}_link">
-      <self_collide>0</self_collide>
-      <enable_wind>0</enable_wind>
-      <kinematic>0</kinematic>
-      <gravity>1</gravity>
-      <!--<mu>1</mu>-->
-      <mu2>1</mu2>
-      <fdir1>0 0 0</fdir1>
-      <!--<slip1>0</slip1>
-      <slip2>0</slip2>-->
-      <kp>1e+13</kp>
-      <kd>1</kd>
-      <!--<max_vel>0.01</max_vel>
-      <min_depth>0</min_depth>-->
-      <sensor name="${name}color" type="camera">
-        <camera name="${name}">
-          <horizontal_fov>${69.4*deg_to_rad}</horizontal_fov>
-          <image>
-            <width>1920</width>
-            <height>1080</height>
-            <format>RGB_INT8</format>
-          </image>
-          <clip>
-            <near>0.1</near>
-            <far>75</far>
-          </clip>
-          <noise>
-            <type>gaussian</type>
-            <mean>0.0</mean>
-            <stddev>0.007</stddev>
-          </noise>
-        </camera>
-        <always_on>true</always_on>
-        <update_rate>30</update_rate>
-        <visualize>true</visualize>
-      </sensor>
-      <sensor name="${name}ired1" type="camera">
-        <camera name="${name}">
-          <horizontal_fov>${85.2*deg_to_rad}</horizontal_fov>
-          <image>
-            <width>1280</width>
-            <height>720</height>
-            <format>L_INT8</format>
-          </image>
-          <clip>
-            <near>0.1</near>
-            <far>75</far>
-          </clip>
-          <noise>
-            <type>gaussian</type>
-            <mean>0.0</mean>
-            <stddev>0.05</stddev>
-          </noise>
-        </camera>
-        <always_on>true</always_on>
-        <update_rate>30</update_rate>
-        <visualize>true</visualize>
-      </sensor>
-      <sensor name="${name}ired2" type="camera">
-        <camera name="${name}">
-          <horizontal_fov>${85.2*deg_to_rad}</horizontal_fov>
-          <image>
-            <width>1280</width>
-            <height>720</height>
-            <format>L_INT8</format>
-          </image>
-          <clip>
-            <near>0.1</near>
-            <far>75</far>
-          </clip>
-          <noise>
-            <type>gaussian</type>
-            <mean>0.0</mean>
-            <stddev>0.05</stddev>
-          </noise>
-        </camera>
-        <always_on>true</always_on>
-        <update_rate>30</update_rate>
-        <visualize>true</visualize>
-      </sensor>
-      <sensor name="${name}depth" type="depth">
-        <camera name="${name}">
-          <horizontal_fov>${85.2*deg_to_rad}</horizontal_fov>
-          <image>
-            <width>1280</width>
-            <height>720</height>
-          </image>
-          <clip>
-            <near>0.1</near>
-            <far>75</far>
-          </clip>
-          <noise>
-            <type>gaussian</type>
-            <mean>0.0</mean>
-            <stddev>0.100</stddev>
-          </noise>
-        </camera>
-        <always_on>true</always_on>
-        <update_rate>30</update_rate>
-        <visualize>true</visualize>
-      </sensor>
-    </gazebo>
-     <gazebo>
-      <plugin name="${name}" filename="librealsense_gazebo_plugin.so">
-        <prefix>${name}</prefix>
-      	<depthUpdateRate>30.0</depthUpdateRate>
-      	<colorUpdateRate>30.0</colorUpdateRate>
-      	<infraredUpdateRate>30.0</infraredUpdateRate>
-      	<depthTopicName>${name}/depth/image_raw</depthTopicName>
-      	<depthCameraInfoTopicName>${name}/depth/camera_info</depthCameraInfoTopicName>
-      	<colorTopicName>${name}/color/image_raw</colorTopicName>
-      	<colorCameraInfoTopicName>${name}/color/camera_info</colorCameraInfoTopicName>
-      	<infrared1TopicName>${name}/infra1/image_raw</infrared1TopicName>
-      	<infrared1CameraInfoTopicName>${name}/infra1/camera_info</infrared1CameraInfoTopicName>
-      	<infrared2TopicName>${name}/infra2/image_raw</infrared2TopicName>
-      	<infrared2CameraInfoTopicName>${name}/infra2/camera_info</infrared2CameraInfoTopicName>
-      	<colorOpticalframeName>${name}_color_optical_frame</colorOpticalframeName>
-      	<depthOpticalframeName>${name}_depth_optical_frame</depthOpticalframeName>
-      	<infrared1OpticalframeName>${name}_infrared1_optical_frame</infrared1OpticalframeName>
-      	<infrared2OpticalframeName>${name}_infrared2_optical_frame</infrared2OpticalframeName>
-      	<rangeMinDepth>0.1</rangeMinDepth>
-      	<rangeMaxDepth>10.0</rangeMaxDepth>
-      	<pointCloud>true</pointCloud>
-      	<pointCloudTopicName>${name}/depth/points</pointCloudTopicName>
-      	<pointCloudCutoff>0.5</pointCloudCutoff>
-      </plugin>
-    </gazebo>
   </xacro:macro>
 </robot>
